File: PCB/PUCKFishProto2Board/proto2board_lay.brd (EAGLE design)
At the start: 66 x 68.2 mm, 13 parts, among them U1 MS583730BA01-50, U2 ZXCT1107SA-7

Commit message: Fixed DRC errors
Changed lines of the file:
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@@
 <wire x1="146.05" y1="68.16170625" x2="144.8562" y2="69.35550625" width="0.4064" layer="1"/>
 <wire x1="144.8562" y1="70.34449375" x2="146.05" y2="71.53829375" width="0.4064" layer="1"/>
-<wire x1="146.05" y1="35.56" x2="146.05" y2="57.15" width="0" layer="19" extent="1-1"/>
 </signal>
 <signal name="MOSI">
@@
 <signal name="!RESET">
 <contactref element="JP2" pad="16"/>
-<wire x1="153.67" y1="97.79" x2="153.543" y2="97.79" width="0.254" layer="1"/>
 </signal>
 <signal name="EN">

Commit message: Fixed angles
Routing:
- net VCC: track 269.9 -> 159.3 mm
- net SDA: track 95.8 -> 154.0 mm
- net A0: track 127.6 -> 107.1 mm
- net N$2: track 76.4 -> 61.6 mm
- net GND: track 130.7 -> 117.8 mm
- net SCL: track 90.6 -> 95.0 mm

Commit message: Latest updates
Routing:
- net VCC: track 159.3 -> 156.0 mm
- net SCL: track 95.0 -> 92.8 mm
- net A0: track 107.1 -> 107.9 mm
- net GND: track 117.8 -> 117.1 mm
Changed lines of the file:
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@@
 <contactref element="RLOAD" pad="1"/>
 <contactref element="RGAIN" pad="2"/>
-<wire x1="107.2144" y1="51.86729375" x2="107.2144" y2="50.27270625" width="0.4064" layer="1"/>
-<wire x1="119.80084375" y1="48.006" x2="120.396" y2="47.41084375" width="0.4064" layer="1"/>
-<wire x1="120.396" y1="47.41084375" x2="120.396" y2="46.56915625" width="0.4064" layer="1"/>
-<wire x1="119.38" y1="45.55315625" x2="119.38" y2="41.91" width="0.4064" layer="1"/>
-<wire x1="120.396" y1="46.56915625" x2="119.38" y2="45.55315625" width="0.4064" layer="1"/>
-<wire x1="107.2144" y1="50.27270625" x2="109.48110625" y2="48.006" width="0.4064" layer="1"/>
-<wire x1="109.48110625" y1="48.006" x2="119.80084375" y2="48.006" width="0.4064" layer="1"/>
-<wire x1="108.22" y1="53.07" x2="108.22" y2="52.87289375" width="0.4064" layer="1"/>
-<wire x1="108.22" y1="52.87289375" x2="107.2144" y2="51.86729375" width="0.4064" layer="1"/>
-<wire x1="127" y1="36.83" x2="123.19" y2="40.64" width="0.4064" layer="1"/>
-<wire x1="123.19" y1="40.64" x2="119.38" y2="40.64" width="0.4064" layer="1"/>
-<wire x1="119.38" y1="40.64" x2="119.38" y2="41.91" width="0.4064" layer="1"/>
 <wire x1="146.05" y1="57.15" x2="146.05" y2="35.56" width="0.4064" layer="16"/>
 <wire x1="146.05" y1="35.56" x2="145.27013125" y2="35.56" width="0.4064" layer="16"/>
@@
 <wire x1="146.05" y1="68.16170625" x2="144.8562" y2="69.35550625" width="0.4064" layer="1"/>
 <wire x1="144.8562" y1="70.34449375" x2="146.05" y2="71.53829375" width="0.4064" layer="1"/>
+<wire x1="127" y1="36.83" x2="124.46" y2="36.83" width="0.4064" layer="1"/>
+<wire x1="124.46" y1="36.83" x2="119.38" y2="41.91" width="0.4064" layer="1"/>
+<wire x1="107.2144" y1="50.27270625" x2="107.2144" y2="51.86729375" width="0.4064" layer="1"/>
+<wire x1="107.98150625" y1="49.5056" x2="107.2144" y2="50.27270625" width="0.4064" layer="1"/>
+<wire x1="118.30124375" y1="49.5056" x2="107.98150625" y2="49.5056" width="0.4064" layer="1"/>
+<wire x1="119.38" y1="41.91" x2="120.396" y2="42.926" width="0.4064" layer="1"/>
+<wire x1="120.396" y1="42.926" x2="120.396" y2="47.41084375" width="0.4064" layer="1"/>
+<wire x1="120.396" y1="47.41084375" x2="118.30124375" y2="49.5056" width="0.4064" layer="1"/>
+<wire x1="108.22" y1="52.87289375" x2="108.22" y2="53.07" width="0.4064" layer="1"/>
+<wire x1="107.2144" y1="51.86729375" x2="108.22" y2="52.87289375" width="0.4064" layer="1"/>
 </signal>
 <signal name="MOSI">
@@
 <wire x1="109.474" y1="65.6844" x2="113.8174" y2="70.0278" width="0.4064" layer="1"/>
 <wire x1="113.8174" y1="70.0278" x2="113.8174" y2="78.1959625" width="0.4064" layer="1"/>
-<wire x1="113.8174" y1="78.1959625" x2="114.8440375" y2="79.2226" width="0.4064" layer="1"/>
-<wire x1="122.4026" y1="79.2226" x2="137.16" y2="93.98" width="0.4064" layer="1"/>
-<wire x1="114.8440375" y1="79.2226" x2="122.4026" y2="79.2226" width="0.4064" layer="1"/>
-<wire x1="137.16" y1="93.98" x2="143.51" y2="93.98" width="0.4064" layer="1"/>
-<wire x1="143.51" y1="93.98" x2="143.51" y2="97.79" width="0.4064" layer="1"/>
+<wire x1="113.8174" y1="78.1959625" x2="125.7914375" y2="90.17" width="0.4064" layer="1"/>
+<wire x1="125.7914375" y1="90.17" x2="140.97" y2="90.17" width="0.4064" layer="1"/>
+<wire x1="140.97" y1="90.17" x2="143.51" y2="92.71" width="0.4064" layer="1"/>
+<wire x1="143.51" y1="92.71" x2="143.51" y2="97.79" width="0.4064" layer="1"/>
 </signal>
 <signal name="PB22/I6/SERCOM5.1">
@@
 <wire x1="118.11" y1="74.93" x2="118.11" y2="77.47" width="0.4064" layer="1"/>
 <wire x1="148.59" y1="35.56" x2="148.59" y2="57.15" width="0.4064" layer="16"/>
-<wire x1="142.2146" y1="56.63446875" x2="141.48553125" y2="55.9054" width="0.4064" layer="16"/>
-<wire x1="141.48553125" y1="55.9054" x2="140.45446875" y2="55.9054" width="0.4064" layer="16"/>
-<wire x1="148.59" y1="57.15" x2="147.3454" y2="58.3946" width="0.4064" layer="16"/>
-<wire x1="147.3454" y1="58.3946" x2="142.99446875" y2="58.3946" width="0.4064" layer="16"/>
-<wire x1="142.99446875" y1="58.3946" x2="142.2146" y2="57.61473125" width="0.4064" layer="16"/>
-<wire x1="142.2146" y1="57.61473125" x2="142.2146" y2="56.63446875" width="0.4064" layer="16"/>
-<wire x1="122.69986875" y1="73.66" x2="118.11" y2="73.66" width="0.4064" layer="16"/>
-<wire x1="140.45446875" y1="55.9054" x2="122.69986875" y2="73.66" width="0.4064" layer="16"/>
-<wire x1="118.11" y1="73.66" x2="118.11" y2="77.47" width="0.4064" layer="16"/>
+<wire x1="146.56553125" y1="58.3946" x2="145.53446875" y2="58.3946" width="0.4064" layer="16"/>
+<wire x1="144.7546" y1="56.63446875" x2="144.02553125" y2="55.9054" width="0.4064" layer="16"/>
+<wire x1="148.59" y1="57.15" x2="147.81013125" y2="57.15" width="0.4064" layer="16"/>
+<wire x1="147.81013125" y1="57.15" x2="146.56553125" y2="58.3946" width="0.4064" layer="16"/>
+<wire x1="145.53446875" y1="58.3946" x2="144.7546" y2="57.61473125" width="0.4064" layer="16"/>
+<wire x1="144.7546" y1="57.61473125" x2="144.7546" y2="56.63446875" width="0.4064" layer="16"/>
+<wire x1="139.6746" y1="55.9054" x2="128.27" y2="67.31" width="0.4064" layer="16"/>
+<wire x1="128.27" y1="67.31" x2="118.11" y2="77.47" width="0.4064" layer="16"/>
+<wire x1="144.02553125" y1="55.9054" x2="139.6746" y2="55.9054" width="0.4064" layer="16"/>
 </signal>
 <signal name="SDA">
@@
 <contactref element="U2" pad="3"/>
 <contactref element="RSENSE" pad="2"/>
-<wire x1="111.01729375" y1="50.0644" x2="111.75289375" y2="50.8" width="0.4064" layer="1"/>
-<wire x1="111.75289375" y1="50.8" x2="127" y2="50.8" width="0.4064" layer="1"/>
-<wire x1="127" y1="50.8" x2="127" y2="46.99" width="0.4064" layer="1"/>
-<wire x1="109.42270625" y1="50.0644" x2="111.01729375" y2="50.0644" width="0.4064" layer="1"/>
 <wire x1="119.3038" y1="77.96449375" x2="118.60449375" y2="78.6638" width="0.4064" layer="1"/>
 <wire x1="115.07550625" y1="78.6638" x2="114.3762" y2="77.96449375" width="0.4064" layer="1"/>
@@
 <wire x1="108.22" y1="51.07" x2="108.41710625" y2="51.07" width="0.4064" layer="1"/>
 <wire x1="108.41710625" y1="51.07" x2="109.42270625" y2="50.0644" width="0.4064" layer="1"/>
-<wire x1="111.75289375" y1="50.8" x2="119.3038" y2="58.35090625" width="0.4064" layer="1"/>
+<wire x1="111.01729375" y1="50.0644" x2="119.3038" y2="58.35090625" width="0.4064" layer="1"/>
 <wire x1="119.3038" y1="58.35090625" x2="119.3038" y2="77.96449375" width="0.4064" layer="1"/>
 <wire x1="114.3762" y1="66.1162" x2="113.03" y2="64.77" width="0.4064" layer="1"/>
 <wire x1="118.60449375" y1="78.6638" x2="115.07550625" y2="78.6638" width="0.4064" layer="1"/>
 <wire x1="113.03" y1="64.77" x2="111.506" y2="64.77" width="0.4064" layer="1"/>
-<wire x1="127" y1="46.99" x2="134.62" y2="54.61" width="0.4064" layer="1"/>
-<wire x1="134.62" y1="54.61" x2="140.97" y2="54.61" width="0.4064" layer="1"/>
-<wire x1="140.97" y1="54.61" x2="140.97" y2="57.15" width="0.4064" layer="1"/>
 <wire x1="127" y1="46.99" x2="130.81" y2="46.99" width="0.4064" layer="1"/>
 <wire x1="130.81" y1="46.99" x2="140.97" y2="36.83" width="0.4064" layer="1"/>
@@
 <wire x1="139.7762" y1="82.6262" x2="151.13" y2="93.98" width="0.4064" layer="16"/>
 <wire x1="151.13" y1="93.98" x2="151.13" y2="97.79" width="0.4064" layer="16"/>
+<wire x1="111.01729375" y1="50.0644" x2="109.42270625" y2="50.0644" width="0.4064" layer="1"/>
+<wire x1="127" y1="46.99" x2="123.9256" y2="50.0644" width="0.4064" layer="1"/>
+<wire x1="123.9256" y1="50.0644" x2="111.01729375" y2="50.0644" width="0.4064" layer="1"/>
+<wire x1="127" y1="46.99" x2="137.16" y2="57.15" width="0.4064" layer="1"/>
+<wire x1="137.16" y1="57.15" x2="140.97" y2="57.15" width="0.4064" layer="1"/>
 </signal>
 <signal name="N$2">
